File: hardware/KiCad/MeetingHub-4/MeetingHub-4.kicad_pcb (KiCad board)
At the start: 2 copper layers, 265 x 160 mm, 70 parts, among them J1 USB-C POWER IN, J2 TRRS Notebook 1, J3 TRRS Notebook 2, J4 TRRS Notebook 3, J5 TRRS Notebook 4, J6 Headset (User), K1 Select NB1, K2 Select NB2, K3 Select NB3, K4 Select NB4, SW1 MUTE, SW2 Select NB1, SW3 Select NB2, SW4 Select NB3, SW5 Select NB4, U1 NE5532, U2 NJM4556A

Commit message: Fix Power/RelayControl net widths and reroute 2 disconnected GND pads
Reduces Power/RelayControl netclass track width from the previous
0.7mm/0.45mm to a uniform 0.3mm (via 0.65mm/0.35mm drill), matching what
was actually applied to the routed copper. This resolves the 5 clearance
errors from the last DRC report, which were all caused by the
over-widened traces crowding neighboring pads.

Also fixes the 2 unconnected_items errors on the GND net. Root cause:
the zone filler splits the GND pour into 3 disjoint copper islands in
this layout (the main plane plus two small isolated pockets around the
U1/mixer area and the C3/C4/R9 area) because the surrounding component
density leaves no legal path for a thermal-relief spoke there. Added a
short stitch trace + via from C3 pin 2 out to open board space that
reaches the main plane; verified no reduction in clearance elsewhere via
a custom pad+track distance check and a clean `kicad-cli pcb export
gerbers` run.

Known remaining issue: U1 pin 4 (GND) and C4 pin 2 (GND) still sit in
their own isolated copper islands, not merged with the main GND plane.
An automated search for a clear stitch path (single- and two-segment,
excluding each part's own sibling pads as false positives) found no
route within safe clearance in either case — both pockets are boxed in
by existing signal traces (e.g. a diagonal NB2_L run cuts across the
open side of C4's pocket). This needs a manual routing pass in the GUI,
where the traces can be seen and threaded around by eye, or a small
layout change to open a path. Please re-run DRC to confirm the fixed
items and get the current state of these 2.
Routing:
- net GND: track 9.89 -> 13.9 mm, vias 5 -> 8

Commit message: Fix R2 unconnected GND pad; restore load-bearing U1 via
Adds a short stitch trace + via from R2 pin 2 (GND) to open board space
that reaches the main GND plane, resolving that unconnected_items error.
Verified with a fresh path search (excluding R2's own sibling pads as
false obstacles) and the pad-inclusive/layer-aware clearance check.

Also removes the redundant via that used to sit directly on C3 pin 2
(same location as the pad, doing nothing since that pin already has a
working stitch to the main plane) but discovered mid-fix that the
equivalent via on U1 pin 4 was NOT redundant — removing it re-isolated
U1 pin 4 from the plane, so it's restored unchanged.

C4 pin 2 (GND) remains unresolved. Ran an A* pathfinding search (not
just angle/distance guessing) from C4's pad out to the main plane,
checking both routing layers, down to a hairline 0.15mm trace, over an
80mm+ radius: no clear path exists at any width. That pocket is fully
enclosed by existing signal traces (NB2_L/R, +5V_AUDIO, and the
resistor-grid routing all wrap around it with no gap). This one needs
either a manual re-route of one of those signal traces in the GUI to
open a path, or a small component shift in a future revision — it isn't
fixable by adding a stitch alone.
Routing:
- net GND: track 13.9 -> 15.9 mm
Changed lines of the file:
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@@
   (segment (start 226.825 230.3019) (end 225.8165 230.3019) (width 0.3) (layer "F.Cu") (net 2))
   (segment (start 186.825 94.9894) (end 186.825 96.75) (width 0.3) (layer "F.Cu") (net 2))
+  (segment (start 111.16 118) (end 109.16 118) (width 0.3) (layer "F.Cu") (net 2))
   (segment (start 226.825 94.9782) (end 226.825 96.75) (width 0.3) (layer "F.Cu") (net 2))
   (segment (start 116 140) (end 120 140) (width 0.3) (layer "F.Cu") (net 2))
@@
   (segment (start 146.825 96.75) (end 146.825 94.9824) (width 0.3) (layer "F.Cu") (net 2))
   (via (at 106.4311 94.9917) (size 0.65) (drill 0.35) (layers "F.Cu" "B.Cu") (net 2))
-  (via (at 116 140) (size 0.65) (drill 0.35) (layers "F.Cu" "B.Cu") (net 2))
+  (via (at 109.16 118) (size 0.65) (drill 0.35) (layers "F.Cu" "B.Cu") (net 2))
   (via (at 120 140) (size 0.65) (drill 0.35) (layers "F.Cu" "B.Cu") (net 2))
   (via (at 226.825 94.9782) (size 0.65) (drill 0.35) (layers "F.Cu" "B.Cu") (net 2))
-  (via (at 75 125.62) (size 0.65) (drill 0.35) (layers "F.Cu" "B.Cu") (net 2))
   (via (at 186.825 94.9894) (size 0.65) (drill 0.35) (layers "F.Cu" "B.Cu") (net 2))
   (via (at 146.825 94.9824) (size 0.65) (drill 0.35) (layers "F.Cu" "B.Cu") (net 2))
+  (via (at 75 125.62) (size 0.65) (drill 0.35) (layers "F.Cu" "B.Cu") (net 2))
   (via (at 225.8165 230.3019) (size 0.65) (drill 0.35) (layers "F.Cu" "B.Cu") (net 2))
   (segment (start 112.8981 140.6107) (end 111.8891 141.6197) (width 0.2) (layer "F.Cu") (net 3))

Commit message: Add 4 mounting holes for enclosure fixing (PCB-001 Fase 3.3.3)
Adds MountingHole_3.2mm_M3 footprints at each corner, 6mm margin from
the board edge, matching the guide's spec. All 4 corners were clear of
other components, so no repositioning was needed. Positions:

  MH1 (66, 91)    - superior esquerdo
  MH2 (319, 91)   - superior direito
  MH3 (66, 239)   - inferior esquerdo
  MH4 (319, 239)  - inferior direito

Updates PCB-001-LayoutGuide.md section 3.3.3 to record the applied
positions instead of just instructions. If the enclosure is already
chosen, these need to line up with its fixing holes/rails before
fabrication - just move the 4 footprints in the GUI if not.
Parts:
- added MH1: MountingHole_3.2mm_M3, MountingHole_3.2mm_M3, F.Cu at (66.0, 91.0)
- added MH2: MountingHole_3.2mm_M3, MountingHole_3.2mm_M3, F.Cu at (319.0, 91.0)
- added MH3: MountingHole_3.2mm_M3, MountingHole_3.2mm_M3, F.Cu at (66.0, 239.0)
- added MH4: MountingHole_3.2mm_M3, MountingHole_3.2mm_M3, F.Cu at (319.0, 239.0)
Changed lines of the file:
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@@
     )
   )
+  (footprint "MountingHole_3.2mm_M3" (layer "F.Cu")
+    (at 66 91)
+    (descr "Mounting Hole 3.2mm, no annular, M3")
+    (tags "mounting hole 3.2mm no annular m3")
+    (attr exclude_from_pos_files exclude_from_bom)
+    (fp_text reference "MH1" (at 0 -4.2) (layer "F.SilkS")
+        (effects (font (size 1 1) (thickness 0.15)))
+    )
+    (fp_text value "MountingHole_3.2mm_M3" (at 0 4.2) (layer "F.Fab")
+        (effects (font (size 1 1) (thickness 0.15)))
+    )
+    (fp_text user "${REFERENCE}" (at 0 0) (layer "F.Fab")
+        (effects (font (size 1 1) (thickness 0.15)))
+    )
+    (fp_circle (center 0 0) (end 3.2 0)
+      (stroke (width 0.15) (type solid)) (fill none) (layer "Cmts.User"))
+    (fp_circle (center 0 0) (end 3.45 0)
+      (stroke (width 0.05) (type solid)) (fill none) (layer "F.CrtYd"))
+    (pad "" np_thru_hole circle (at 0 0) (size 3.2 3.2) (drill 3.2) (layers "*.Cu" "*.Mask"))
+  )
   (footprint "Resistor_THT:R_Axial_DIN0207_L6.3mm_D2.5mm_P10.16mm_Horizontal" (layer "F.Cu")
     (at 75 140)
@@
     )
   )
+  (footprint "MountingHole_3.2mm_M3" (layer "F.Cu")
+    (at 319 239)
+    (descr "Mounting Hole 3.2mm, no annular, M3")
+    (tags "mounting hole 3.2mm no annular m3")
+    (attr exclude_from_pos_files exclude_from_bom)
+    (fp_text reference "MH4" (at 0 -4.2) (layer "F.SilkS")
+        (effects (font (size 1 1) (thickness 0.15)))
+    )
+    (fp_text value "MountingHole_3.2mm_M3" (at 0 4.2) (layer "F.Fab")
+        (effects (font (size 1 1) (thickness 0.15)))
+    )
+    (fp_text user "${REFERENCE}" (at 0 0) (layer "F.Fab")
+        (effects (font (size 1 1) (thickness 0.15)))
+    )
+    (fp_circle (center 0 0) (end 3.2 0)
+      (stroke (width 0.15) (type solid)) (fill none) (layer "Cmts.User"))
+    (fp_circle (center 0 0) (end 3.45 0)
+      (stroke (width 0.05) (type solid)) (fill none) (layer "F.CrtYd"))
+    (pad "" np_thru_hole circle (at 0 0) (size 3.2 3.2) (drill 3.2) (layers "*.Cu" "*.Mask"))
+  )
   (footprint "Capacitor_THT:C_Disc_D5.0mm_W2.5mm_P2.50mm" (layer "F.Cu")
     (at 101 162)
@@
     )
   )
+  (footprint "MountingHole_3.2mm_M3" (layer "F.Cu")
+    (at 319 91)
+    (descr "Mounting Hole 3.2mm, no annular, M3")
+    (tags "mounting hole 3.2mm no annular m3")
+    (attr exclude_from_pos_files exclude_from_bom)
+    (fp_text reference "MH2" (at 0 -4.2) (layer "F.SilkS")
+        (effects (font (size 1 1) (thickness 0.15)))
+    )
+    (fp_text value "MountingHole_3.2mm_M3" (at 0 4.2) (layer "F.Fab")
+        (effects (font (size 1 1) (thickness 0.15)))
+    )
+    (fp_text user "${REFERENCE}" (at 0 0) (layer "F.Fab")
+        (effects (font (size 1 1) (thickness 0.15)))
+    )
+    (fp_circle (center 0 0) (end 3.2 0)
+      (stroke (width 0.15) (type solid)) (fill none) (layer "Cmts.User"))
+    (fp_circle (center 0 0) (end 3.45 0)
+      (stroke (width 0.05) (type solid)) (fill none) (layer "F.CrtYd"))
+    (pad "" np_thru_hole circle (at 0 0) (size 3.2 3.2) (drill 3.2) (layers "*.Cu" "*.Mask"))
+  )
   (footprint "Resistor_THT:R_Axial_DIN0207_L6.3mm_D2.5mm_P10.16mm_Horizontal" (layer "F.Cu")
     (at 101 140)
@@
     )
   )
+  (footprint "MountingHole_3.2mm_M3" (layer "F.Cu")
+    (at 66 239)
+    (descr "Mounting Hole 3.2mm, no annular, M3")
+    (tags "mounting hole 3.2mm no annular m3")
+    (attr exclude_from_pos_files exclude_from_bom)
+    (fp_text reference "MH3" (at 0 -4.2) (layer "F.SilkS")
+        (effects (font (size 1 1) (thickness 0.15)))
+    )
+    (fp_text value "MountingHole_3.2mm_M3" (at 0 4.2) (layer "F.Fab")
+        (effects (font (size 1 1) (thickness 0.15)))
+    )
+    (fp_text user "${REFERENCE}" (at 0 0) (layer "F.Fab")
+        (effects (font (size 1 1) (thickness 0.15)))
+    )
+    (fp_circle (center 0 0) (end 3.2 0)
+      (stroke (width 0.15) (type solid)) (fill none) (layer "Cmts.User"))
+    (fp_circle (center 0 0) (end 3.45 0)
+      (stroke (width 0.05) (type solid)) (fill none) (layer "F.CrtYd"))
+    (pad "" np_thru_hole circle (at 0 0) (size 3.2 3.2) (drill 3.2) (layers "*.Cu" "*.Mask"))
+  )
   (gr_line (start 60 85) (end 325 85)

Commit message: Fix missing library reference on MH1-4 mounting holes
The mounting holes added for Fase 3.3.3 were inserted via a direct
filesystem path load (pcbnew.FootprintLoad), which left their FPID
without a library nickname - saved as bare "MountingHole_3.2mm_M3"
instead of "MountingHole:MountingHole_3.2mm_M3". DRC caught this as
[lib_footprint_issues]: "library ''" on all 4. Fixed by setting the
correct LIB_ID (library nickname "MountingHole", matching the global
fp-lib-table entry for MountingHole.pretty). Verified gerber export
still succeeds.
Parts:
- MH1, MH2, MH3, MH4: footprint MountingHole_3.2mm_M3 -> MountingHole:MountingHole_3.2mm_M3
Changed lines of the file:
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@@
     )
   )
-  (footprint "MountingHole_3.2mm_M3" (layer "F.Cu")
+  (footprint "MountingHole:MountingHole_3.2mm_M3" (layer "F.Cu")
     (at 66 91)
     (descr "Mounting Hole 3.2mm, no annular, M3")
@@
     )
   )
-  (footprint "MountingHole_3.2mm_M3" (layer "F.Cu")
+  (footprint "MountingHole:MountingHole_3.2mm_M3" (layer "F.Cu")
     (at 319 239)
     (descr "Mounting Hole 3.2mm, no annular, M3")
@@
     )
   )
-  (footprint "MountingHole_3.2mm_M3" (layer "F.Cu")
+  (footprint "MountingHole:MountingHole_3.2mm_M3" (layer "F.Cu")
     (at 319 91)
     (descr "Mounting Hole 3.2mm, no annular, M3")
@@
     )
   )
-  (footprint "MountingHole_3.2mm_M3" (layer "F.Cu")
+  (footprint "MountingHole:MountingHole_3.2mm_M3" (layer "F.Cu")
     (at 66 239)
     (descr "Mounting Hole 3.2mm, no annular, M3")

Commit message: Versao pre final
Routing:
- net +5V_AUDIO: track 485.5 -> 490.9 mm
- net GND: track 15.9 -> 19.8 mm, vias 8 -> 9
Changed lines of the file:
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@@
   (segment (start 258.117 219.883) (end 221.5125 219.883) (width 0.3) (layer "F.Cu") (net 1))
   (segment (start 174.6981 233.3019) (end 176 232) (width 0.3) (layer "F.Cu") (net 1))
+  (segment (start 189.270243 134.62) (end 132.38 134.62) (width 0.3) (layer "F.Cu") (net 1))
   (segment (start 287.7962 133.8981) (end 271.1019 133.8981) (width 0.3) (layer "F.Cu") (net 1))
   (segment (start 290 135) (end 288.8981 135) (width 0.3) (layer "F.Cu") (net 1))
   (segment (start 82.62 118) (end 88 118) (width 0.3) (layer "F.Cu") (net 1))
   (segment (start 195.3538 233.3538) (end 194 232) (width 0.3) (layer "F.Cu") (net 1))
+  (segment (start 196.890243 142.24) (end 189.270243 134.62) (width 0.3) (layer "F.Cu") (net 1))
   (segment (start 260 218) (end 258.117 219.883) (width 0.3) (layer "F.Cu") (net 1))
   (segment (start 127 140) (end 123.3029 136.3029) (width 0.3) (layer "F.Cu") (net 1))
   (segment (start 192.6981 233.3019) (end 194 232) (width 0.3) (layer "F.Cu") (net 1))
+  (segment (start 262.76 142.24) (end 196.890243 142.24) (width 0.3) (layer "F.Cu") (net 1))
+  (segment (start 270 135) (end 262.76 142.24) (width 0.3) (layer "F.Cu") (net 1))
   (segment (start 123.3029 136.3029) (end 116.8571 136.3029) (width 0.3) (layer "F.Cu") (net 1))
   (segment (start 177.3019 233.3019) (end 192.6981 233.3019) (width 0.3) (layer "F.Cu") (net 1))
-  (segment (start 270 135) (end 263.8847 141.1153) (width 0.3) (layer "F.Cu") (net 1))
   (segment (start 159.3019 233.3019) (end 174.6981 233.3019) (width 0.3) (layer "F.Cu") (net 1))
+  (segment (start 132.38 134.62) (end 127 140) (width 0.3) (layer "F.Cu") (net 1))
   (segment (start 271.1019 133.8981) (end 270 135) (width 0.3) (layer "F.Cu") (net 1))
-  (segment (start 128.115299 141.1153) (end 127 140) (width 0.3) (layer "F.Cu") (net 1))
   (segment (start 176 232) (end 177.3019 233.3019) (width 0.3) (layer "F.Cu") (net 1))
   (segment (start 210.6462 233.3538) (end 195.3538 233.3538) (width 0.3) (layer "F.Cu") (net 1))
   (segment (start 288.8981 135) (end 287.7962 133.8981) (width 0.3) (layer "F.Cu") (net 1))
-  (segment (start 263.8847 141.1153) (end 128.115299 141.1153) (width 0.3) (layer "F.Cu") (net 1))
   (via (at 221.5125 219.883) (size 0.65) (drill 0.35) (layers "F.Cu" "B.Cu") (net 1))
   (via (at 116.8571 136.3029) (size 0.65) (drill 0.35) (layers "F.Cu" "B.Cu") (net 1))
@@
   (segment (start 212 232) (end 213.3311 233.3311) (width 0.3) (layer "B.Cu") (net 1))
   (segment (start 106.6375 95.1981) (end 106.4311 94.9917) (width 0.3) (layer "F.Cu") (net 2))
+  (segment (start 132.08 137.42) (end 129.5 140) (width 0.3) (layer "F.Cu") (net 2))
+  (segment (start 132.08 137.16) (end 132.08 137.42) (width 0.3) (layer "F.Cu") (net 2))
   (segment (start 106.825 95.1981) (end 106.6375 95.1981) (width 0.3) (layer "F.Cu") (net 2))
   (segment (start 106.825 96.75) (end 106.825 95.1981) (width 0.3) (layer "F.Cu") (net 2))
@@
   (segment (start 111.16 118) (end 109.16 118) (width 0.3) (layer "F.Cu") (net 2))
   (segment (start 226.825 94.9782) (end 226.825 96.75) (width 0.3) (layer "F.Cu") (net 2))
+  (segment (start 226.825 228.75) (end 226.825 230.3019) (width 0.3) (layer "F.Cu") (net 2))
   (segment (start 116 140) (end 120 140) (width 0.3) (layer "F.Cu") (net 2))
-  (segment (start 226.825 228.75) (end 226.825 230.3019) (width 0.3) (layer "F.Cu") (net 2))
   (segment (start 146.825 96.75) (end 146.825 94.9824) (width 0.3) (layer "F.Cu") (net 2))
   (via (at 106.4311 94.9917) (size 0.65) (drill 0.35) (layers "F.Cu" "B.Cu") (net 2))
@@
   (via (at 75 125.62) (size 0.65) (drill 0.35) (layers "F.Cu" "B.Cu") (net 2))
   (via (at 225.8165 230.3019) (size 0.65) (drill 0.35) (layers "F.Cu" "B.Cu") (net 2))
+  (via (at 132.08 137.16) (size 0.65) (drill 0.35) (layers "F.Cu" "B.Cu") (net 2))
   (segment (start 112.8981 140.6107) (end 111.8891 141.6197) (width 0.2) (layer "F.Cu") (net 3))
   (segment (start 192.5 175) (end 190 175) (width 0.2) (layer "F.Cu") (net 3))
