File: hardware/KiCad/MeetingHub-4/MeetingHub-4.kicad_pcb (KiCad board)
At the start: 4 copper layers, 265 x 160 mm, 75 parts, among them J1 USB-C POWER IN, J2 TRRS Notebook 1, J3 TRRS Notebook 2, J4 TRRS Notebook 3, J5 TRRS Notebook 4, J6 Headset (User), K1 Select NB1, K2 Select NB2, K3 Select NB3, K4 Select NB4, SW1 MUTE, SW2 Select NB1, SW3 Select NB2, SW4 Select NB3, SW5 Select NB4, U1 NE5532, U2 NJM4556A

Commit message: Fix real ERC errors: TP1 never connected, U1 power_pin_not_driven, stale AudioJack4 lib_id
- POWER.kicad_sch: add missing junction so TP1 actually joins the
  +5V_AUDIO wire (visual overlap without a junction is not a real
  connection in KiCad); add two power:PWR_FLAG symbols (+5V_AUDIO, GND)
  so ERC has an explicit power source for nets fed only by J1's USB-C
  VBUS pin, resolving power_pin_not_driven on U1.
- MeetingHub-4.kicad_pcb: TP1's pad had no net at all on the physical
  board (unconnected-(TP1-Pad1)), and TP2 (GND test point added
  directly on the PCB) had no net either - both test points were
  floating on the real board despite BOM/docs claiming otherwise. Fixed
  by assigning TP1 to +5V_AUDIO and TP2 to GND, then refilling the
  internal planes so the pads actually bond to them. Verified 0
  unconnected items and 0 real DRC errors after the fix.
- TRRS.kicad_sch: J2-J6 referenced Connector:AudioJack4, a library path
  that no longer exists in current KiCad (symbol moved to
  Connector_Audio) - only worked because of the cached copy. Repointed
  lib_id to Connector_Audio:AudioJack4 after confirming the cached
  symbol is byte-identical to the current system library version.

Found while working through the user's real GUI ERC report (248
messages). Documented in PCB-001 Fase 11 and BOM-002-AsBuilt Seção 4.

Co-Authored-By: Claude Sonnet 5 <noreply@anthropic.com>
Connections:
- TP1 pad 1: unconnected-(TP1-Pad1) -> +5V_AUDIO
- TP2 pad 1: (no net) -> GND
Changed lines of the file:
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@@
   (net 70 "Net-(U2A--)")
   (net 71 "Net-(U2B--)")
-  (net 72 "unconnected-(TP1-Pad1)")
   (footprint "Connector_Audio:Jack_3.5mm_PJ320D_Horizontal" (layer "F.Cu")
     (at 150 100)
@@
     (fp_circle (center 0 0) (end 1.25 0)
       (stroke (width 0.05) (type solid)) (fill none) (layer "F.CrtYd"))
-    (pad "1" thru_hole circle (at 0 0) (size 1.5 1.5) (drill 0.7) (layers "*.Cu" "*.Mask"))
+    (pad "1" thru_hole circle (at 0 0) (size 1.5 1.5) (drill 0.7) (layers "*.Cu" "*.Mask")
+      (net 2 "GND"))
   )
   (footprint "Connector_Audio:Jack_3.5mm_PJ320D_Horizontal" (layer "F.Cu")
@@
       (stroke (width 0.05) (type solid)) (fill none) (layer "F.CrtYd"))
     (pad "1" thru_hole circle (at 0 0) (size 1.5 1.5) (drill 0.7) (layers "*.Cu" "*.Mask")
-      (net 72 "unconnected-(TP1-Pad1)") (pinfunction "1") (pintype "passive"))
+      (net 1 "+5V_AUDIO") (pinfunction "1") (pintype "passive"))
   )
   (footprint "Resistor_THT:R_Axial_DIN0207_L6.3mm_D2.5mm_P10.16mm_Horizontal" (layer "F.Cu")
