File: hardware/KiCad/MeetingHub-4/TRRS.kicad_sch (KiCad schematic)
At the start: 4 parts, among them J2 TRRS Notebook 1, J3 TRRS Notebook 2, J4 TRRS Notebook 3, J5 TRRS Notebook 4

Commit message: Fix real ERC errors: TP1 never connected, U1 power_pin_not_driven, stale AudioJack4 lib_id
- POWER.kicad_sch: add missing junction so TP1 actually joins the
  +5V_AUDIO wire (visual overlap without a junction is not a real
  connection in KiCad); add two power:PWR_FLAG symbols (+5V_AUDIO, GND)
  so ERC has an explicit power source for nets fed only by J1's USB-C
  VBUS pin, resolving power_pin_not_driven on U1.
- MeetingHub-4.kicad_pcb: TP1's pad had no net at all on the physical
  board (unconnected-(TP1-Pad1)), and TP2 (GND test point added
  directly on the PCB) had no net either - both test points were
  floating on the real board despite BOM/docs claiming otherwise. Fixed
  by assigning TP1 to +5V_AUDIO and TP2 to GND, then refilling the
  internal planes so the pads actually bond to them. Verified 0
  unconnected items and 0 real DRC errors after the fix.
- TRRS.kicad_sch: J2-J6 referenced Connector:AudioJack4, a library path
  that no longer exists in current KiCad (symbol moved to
  Connector_Audio) - only worked because of the cached copy. Repointed
  lib_id to Connector_Audio:AudioJack4 after confirming the cached
  symbol is byte-identical to the current system library version.

Found while working through the user's real GUI ERC report (248
messages). Documented in PCB-001 Fase 11 and BOM-002-AsBuilt Seção 4.

Co-Authored-By: Claude Sonnet 5 <noreply@anthropic.com>
Parts:
- J2, J3, J4, J5: symbol Connector:AudioJack4 -> Connector_Audio:AudioJack4
Changed lines of the file:
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@@
     )
   )
-  (symbol (lib_id "Connector:AudioJack4") (at 50 78 0) (unit 1)
+  (symbol (lib_id "Connector_Audio:AudioJack4") (at 50 78 0) (unit 1)
     (in_bom yes) (on_board yes) (dnp no)
     (property "Reference" "J3" (at 50 71.65 0)
@@
     )
   )
-  (symbol (lib_id "Connector:AudioJack4") (at 50 154 0) (unit 1)
+  (symbol (lib_id "Connector_Audio:AudioJack4") (at 50 154 0) (unit 1)
     (in_bom yes) (on_board yes) (dnp no)
     (property "Reference" "J5" (at 50 147.65 0)
@@
     )
   )
-  (symbol (lib_id "Connector:AudioJack4") (at 50 40 0) (unit 1)
+  (symbol (lib_id "Connector_Audio:AudioJack4") (at 50 40 0) (unit 1)
     (in_bom yes) (on_board yes) (dnp no)
     (property "Reference" "J2" (at 50 33.65 0)
@@
     )
   )
-  (symbol (lib_id "Connector:AudioJack4") (at 50 116 0) (unit 1)
+  (symbol (lib_id "Connector_Audio:AudioJack4") (at 50 116 0) (unit 1)
     (in_bom yes) (on_board yes) (dnp no)
     (property "Reference" "J4" (at 50 109.65 0)
