File: hardware/KiCad/MeetingHub-4/HPAMP.kicad_sch (KiCad schematic)
At the start: 17 parts, among them J6 Headset (User), U2 NJM4556A

Commit message: Fix remaining ERC errors: wrong PWR_FLAG net, missing no-connects, J6 AudioJack4
- POWER.kicad_sch: relocate #FLG01 (+5V_AUDIO PWR_FLAG) - it was tapped
  on the wire feeding fuse F1 from the input side, not the actual
  +5V_AUDIO net downstream of F1 (same node as TP1 and the +5V_AUDIO
  global label). U1 Pin 8 (V+) kept reporting power_pin_not_driven
  because of this even after the first fix. Also add no_connect markers
  on J1's 9 unused USB-C pins (D+, D-, CC1, CC2, SBU1, SBU2, SHIELD) -
  intentional since J1 is power-only, but ERC flagged them as errors
  without an explicit no-connect.
- MICSW.kicad_sch: add no_connect on K1-K4 pin 10 (duplicate reverse
  relay contact, unused in this SPDT wiring) - same reasoning, silences
  a real ERC error instead of just being documented as expected.
- HPAMP.kicad_sch: J6 also referenced the stale Connector:AudioJack4
  lib_id (missed in the previous fix, which only covered J2-J5 in
  TRRS.kicad_sch). Repointed to Connector_Audio:AudioJack4.

Found from the user's second real ERC report after the previous round
of fixes. Documented in PCB-001 Fase 11 and BOM-002-AsBuilt Seção 4.

Co-Authored-By: Claude Sonnet 5 <noreply@anthropic.com>
Parts:
- J6: symbol Connector:AudioJack4 -> Connector_Audio:AudioJack4
Changed lines of the file:
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@@
     )
   )
-  (symbol (lib_id "Connector:AudioJack4") (at 200 60 0) (unit 1)
+  (symbol (lib_id "Connector_Audio:AudioJack4") (at 200 60 0) (unit 1)
     (in_bom yes) (on_board yes) (dnp no)
     (property "Reference" "J6" (at 200 53.65 0)
