File: hardware/KiCad/MeetingHub-4/HPAMP.kicad_sch (KiCad schematic)
At the start: 17 parts, among them J6 Headset (User), U2 NJM4556A

Commit message: jlcpcb production  W2026080810364558  PCB/PCBA
Parts:
- C21: footprint Capacitor_THT:C_Disc_D5.0mm_W2.5mm_P2.50mm -> Capacitor_SMD:C_0603_1608Metric
Changed lines of the file:
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@@
       (effects (font (size 1.27 1.27)))
     )
-    (property "Footprint" "Capacitor_THT:C_Disc_D5.0mm_W2.5mm_P2.50mm" (at 129.54 15.24 0)
+    (property "Footprint" "Capacitor_SMD:C_0603_1608Metric" (at 129.54 15.24 0)
       (effects (font (size 1.27 1.27)) hide)
     )
