File: hardware/KiCad/MeetingHub-4/MICSW.kicad_sch (KiCad schematic)
At the start: 13 parts, among them K1 Select NB1, K2 Select NB2, K3 Select NB3, K4 Select NB4, SW1 MUTE, SW2 Select NB1, SW3 Select NB2, SW4 Select NB3, SW5 Select NB4

Commit message: Fix remaining ERC errors: wrong PWR_FLAG net, missing no-connects, J6 AudioJack4
- POWER.kicad_sch: relocate #FLG01 (+5V_AUDIO PWR_FLAG) - it was tapped
  on the wire feeding fuse F1 from the input side, not the actual
  +5V_AUDIO net downstream of F1 (same node as TP1 and the +5V_AUDIO
  global label). U1 Pin 8 (V+) kept reporting power_pin_not_driven
  because of this even after the first fix. Also add no_connect markers
  on J1's 9 unused USB-C pins (D+, D-, CC1, CC2, SBU1, SBU2, SHIELD) -
  intentional since J1 is power-only, but ERC flagged them as errors
  without an explicit no-connect.
- MICSW.kicad_sch: add no_connect on K1-K4 pin 10 (duplicate reverse
  relay contact, unused in this SPDT wiring) - same reasoning, silences
  a real ERC error instead of just being documented as expected.
- HPAMP.kicad_sch: J6 also referenced the stale Connector:AudioJack4
  lib_id (missed in the previous fix, which only covered J2-J5 in
  TRRS.kicad_sch). Repointed to Connector_Audio:AudioJack4.

Found from the user's second real ERC report after the previous round
of fixes. Documented in PCB-001 Fase 11 and BOM-002-AsBuilt Seção 4.

Co-Authored-By: Claude Sonnet 5 <noreply@anthropic.com>
Connections:
- no-connect marks 0 -> 4
Changed lines of the file:
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@@
     (stroke (width 0) (type default))
   )
+  (no_connect (at 127.62 52.38))
+  (no_connect (at 127.62 92.38))
+  (no_connect (at 127.62 132.38))
+  (no_connect (at 127.62 172.38))
   (wire (pts (xy 114.92 107.62) (xy 127.62 107.62))
     (stroke (width 0) (type default))
