File: hardware/KiCad/MeetingHub-4/POWER.kicad_sch (KiCad schematic)
At the start: 6 parts, among them J1 USB-C POWER IN

Commit message: jlcpcb production  W2026080810364558  PCB/PCBA
Parts:
- C1: footprint Capacitor_THT:C_Disc_D5.0mm_W2.5mm_P2.50mm -> Capacitor_SMD:C_0603_1608Metric
- D1: footprint Diode_THT:D_DO-41_SOD81_P10.16mm_Horizontal -> Diode_SMD:Nexperia_DSN1608-2_1.6x0.8mm
Changed lines of the file:
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@@
       (effects (font (size 1.27 1.27)) (justify left))
     )
-    (property "Footprint" "Capacitor_THT:C_Disc_D5.0mm_W2.5mm_P2.50mm" (at 79.7052 64.77 0)
+    (property "Footprint" "Capacitor_SMD:C_0603_1608Metric" (at 79.7052 64.77 0)
       (effects (font (size 1.27 1.27)) hide)
     )
@@
       (effects (font (size 1.27 1.27)))
     )
-    (property "Footprint" "Diode_THT:D_DO-41_SOD81_P10.16mm_Horizontal" (at 66.04 66.04 0)
+    (property "Footprint" "Diode_SMD:Nexperia_DSN1608-2_1.6x0.8mm" (at 66.04 66.04 0)
       (effects (font (size 1.27 1.27)) hide)
     )
