File: hardware/KiCad/MeetingHub-4/MIXER.kicad_sch (KiCad schematic)
At the start: 30 parts, among them U1 NE5532

Commit message: Resize and relayout
Parts:
- RV1, RV2, RV3, RV4: footprint Potentiometer_THT:Potentiometer_Alps_RK097_Dual_Horizontal -> Connector_JST:JST_XH_B6B-XH-A_1x06_P2.50mm_Vertical
- RV5: footprint Potentiometer_THT:Potentiometer_Alps_RK097_Dual_Horizontal -> Connector_JST:JST_XH_S6B-XH-A_1x06_P2.50mm_Horizontal
Changed lines of the file:
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@@
       (effects (font (size 1.27 1.27)))
     )
-    (property "Footprint" "Potentiometer_THT:Potentiometer_Alps_RK097_Dual_Horizontal" (at 85.09 133.35 0)
+    (property "Footprint" "Connector_JST:JST_XH_B6B-XH-A_1x06_P2.50mm_Vertical" (at 85.09 133.35 0)
       (effects (font (size 1.27 1.27)) hide)
     )
@@
       (effects (font (size 1.27 1.27)))
     )
-    (property "Footprint" "Potentiometer_THT:Potentiometer_Alps_RK097_Dual_Horizontal" (at 279.4 90.17 0)
+    (property "Footprint" "Connector_JST:JST_XH_S6B-XH-A_1x06_P2.50mm_Horizontal" (at 279.4 90.17 0)
       (effects (font (size 1.27 1.27)) hide)
     )
@@
       (effects (font (size 1.27 1.27)))
     )
-    (property "Footprint" "Potentiometer_THT:Potentiometer_Alps_RK097_Dual_Horizontal" (at 85.09 99.06 0)
+    (property "Footprint" "Connector_JST:JST_XH_B6B-XH-A_1x06_P2.50mm_Vertical" (at 85.09 99.06 0)
       (effects (font (size 1.27 1.27)) hide)
     )
@@
       (effects (font (size 1.27 1.27)))
     )
-    (property "Footprint" "Potentiometer_THT:Potentiometer_Alps_RK097_Dual_Horizontal" (at 85.09 166.37 0)
+    (property "Footprint" "Connector_JST:JST_XH_B6B-XH-A_1x06_P2.50mm_Vertical" (at 85.09 166.37 0)
       (effects (font (size 1.27 1.27)) hide)
     )
@@
       (effects (font (size 1.27 1.27)))
     )
-    (property "Footprint" "Potentiometer_THT:Potentiometer_Alps_RK097_Dual_Horizontal" (at 85.09 64.77 0)
-      (effects (font (size 1.27 1.27)) hide)
-    )
+    (property "Footprint" "Connector_JST:JST_XH_B6B-XH-A_1x06_P2.50mm_Vertical" (at 85.09 64.77 0)
+      (effects (font (size 1.27 1.27)) hide)
+    )

Commit message: jlcpcb production  W2026080810364558  PCB/PCBA
Parts:
- C4: footprint Capacitor_THT:C_Disc_D5.0mm_W2.5mm_P2.50mm -> Capacitor_SMD:C_0603_1608Metric
- RV1, RV2, RV3, RV4: footprint Connector_JST:JST_XH_B6B-XH-A_1x06_P2.50mm_Vertical -> MeetingHub-4:Potentiometer_Alps_RK09L_Double_Vertical
- RV5: footprint Connector_JST:JST_XH_S6B-XH-A_1x06_P2.50mm_Horizontal -> Potentiometer_THT:Potentiometer_Alps_RK097_Dual_Horizontal
Changed lines of the file:
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@@
       (effects (font (size 1.27 1.27)))
     )
-    (property "Footprint" "Connector_JST:JST_XH_B6B-XH-A_1x06_P2.50mm_Vertical" (at 85.09 133.35 0)
+    (property "Footprint" "MeetingHub-4:Potentiometer_Alps_RK09L_Double_Vertical" (at 85.09 133.35 0)
       (effects (font (size 1.27 1.27)) hide)
     )
@@
       (effects (font (size 1.27 1.27)))
     )
-    (property "Footprint" "Connector_JST:JST_XH_S6B-XH-A_1x06_P2.50mm_Horizontal" (at 279.4 90.17 0)
+    (property "Footprint" "Potentiometer_THT:Potentiometer_Alps_RK097_Dual_Horizontal" (at 279.4 90.17 0)
       (effects (font (size 1.27 1.27)) hide)
     )
@@
       (effects (font (size 1.27 1.27)))
     )
-    (property "Footprint" "Capacitor_THT:C_Disc_D5.0mm_W2.5mm_P2.50mm" (at 80.01 25.4 0)
+    (property "Footprint" "Capacitor_SMD:C_0603_1608Metric" (at 80.01 25.4 0)
       (effects (font (size 1.27 1.27)) hide)
     )
@@
       (effects (font (size 1.27 1.27)))
     )
-    (property "Footprint" "Connector_JST:JST_XH_B6B-XH-A_1x06_P2.50mm_Vertical" (at 85.09 99.06 0)
+    (property "Footprint" "MeetingHub-4:Potentiometer_Alps_RK09L_Double_Vertical" (at 85.09 99.06 0)
       (effects (font (size 1.27 1.27)) hide)
     )
@@
       (effects (font (size 1.27 1.27)))
     )
-    (property "Footprint" "Connector_JST:JST_XH_B6B-XH-A_1x06_P2.50mm_Vertical" (at 85.09 166.37 0)
+    (property "Footprint" "MeetingHub-4:Potentiometer_Alps_RK09L_Double_Vertical" (at 85.09 166.37 0)
       (effects (font (size 1.27 1.27)) hide)
     )
@@
       (effects (font (size 1.27 1.27)))
     )
-    (property "Footprint" "Connector_JST:JST_XH_B6B-XH-A_1x06_P2.50mm_Vertical" (at 85.09 64.77 0)
-      (effects (font (size 1.27 1.27)) hide)
-    )
+    (property "Footprint" "MeetingHub-4:Potentiometer_Alps_RK09L_Double_Vertical" (at 85.09 64.77 0)
+      (effects (font (size 1.27 1.27)) hide)
+    )

Commit message: Rascunho projeto após fabricação com prblemas
Connections:
- net VBIAS: now also RV1.1, RV1.4, RV2.1, RV2.4, RV3.1, RV3.4, RV4.1, RV4.4, RV5.1, RV5.4; no longer RV1.3, RV1.6, RV2.3, RV2.6, RV3.3, RV3.6, RV4.3, RV4.6, RV5.3, RV5.6
- net at C11.2: now also RV4.3; no longer RV4.1
- net at C14.2: now also RV5.6; no longer RV5.4
- net at C8.2: now also RV2.6; no longer RV2.4
- net at C7.2: now also RV2.3; no longer RV2.1
- net at C9.2: now also RV3.3; no longer RV3.1
- net at C10.2: now also RV3.6; no longer RV3.4
- net at C13.2: now also RV5.3; no longer RV5.1
- net at C6.2: now also RV1.6; no longer RV1.4
- net at C12.2: now also RV4.6; no longer RV4.4
- net at C5.2: now also RV1.3; no longer RV1.1
Changed lines of the file:
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@@
     (stroke (width 0) (type default))
   )
-  (wire (pts (xy 54.61 144.78) (xy 87.63 135.89))
-    (stroke (width 0) (type default))
-  )
-  (wire (pts (xy 255.27 114.3) (xy 281.94 92.71))
+  (wire (pts (xy 54.61 144.78) (xy 95.25 135.89))
+    (stroke (width 0) (type default))
+  )
+  (wire (pts (xy 255.27 114.3) (xy 289.56 92.71))
     (stroke (width 0) (type default))
   )
@@
     (stroke (width 0) (type default))
   )
-  (wire (pts (xy 82.55 135.89) (xy 82.55 129.54))
-    (stroke (width 0) (type default))
-  )
-  (wire (pts (xy 95.25 67.31) (xy 95.25 60.96))
+  (wire (pts (xy 74.93 135.89) (xy 74.93 129.54))
+    (stroke (width 0) (type default))
+  )
+  (wire (pts (xy 87.63 67.31) (xy 87.63 60.96))
     (stroke (width 0) (type default))
   )
@@
     (stroke (width 0) (type default))
   )
-  (wire (pts (xy 54.61 162.56) (xy 74.93 168.91))
+  (wire (pts (xy 54.61 162.56) (xy 82.55 168.91))
     (stroke (width 0) (type default))
   )
@@
     (stroke (width 0) (type default))
   )
-  (wire (pts (xy 82.55 168.91) (xy 82.55 162.56))
+  (wire (pts (xy 74.93 168.91) (xy 74.93 162.56))
     (stroke (width 0) (type default))
   )
@@
     (stroke (width 0) (type default))
   )
-  (wire (pts (xy 54.61 179.07) (xy 87.63 168.91))
+  (wire (pts (xy 54.61 179.07) (xy 95.25 168.91))
     (stroke (width 0) (type default))
   )
@@
     (stroke (width 0) (type default))
   )
-  (wire (pts (xy 95.25 101.6) (xy 95.25 95.25))
+  (wire (pts (xy 87.63 101.6) (xy 87.63 95.25))
     (stroke (width 0) (type default))
   )
@@
     (stroke (width 0) (type default))
   )
-  (wire (pts (xy 54.61 76.2) (xy 87.63 67.31))
-    (stroke (width 0) (type default))
-  )
-  (wire (pts (xy 82.55 67.31) (xy 82.55 60.96))
-    (stroke (width 0) (type default))
-  )
-  (wire (pts (xy 276.86 92.71) (xy 276.86 85.09))
-    (stroke (width 0) (type default))
-  )
-  (wire (pts (xy 54.61 128.27) (xy 74.93 135.89))
-    (stroke (width 0) (type default))
-  )
-  (wire (pts (xy 95.25 135.89) (xy 95.25 129.54))
-    (stroke (width 0) (type default))
-  )
-  (wire (pts (xy 82.55 101.6) (xy 82.55 95.25))
+  (wire (pts (xy 54.61 76.2) (xy 95.25 67.31))
+    (stroke (width 0) (type default))
+  )
+  (wire (pts (xy 74.93 67.31) (xy 74.93 60.96))
+    (stroke (width 0) (type default))
+  )
+  (wire (pts (xy 269.24 92.71) (xy 269.24 85.09))
+    (stroke (width 0) (type default))
+  )
+  (wire (pts (xy 54.61 128.27) (xy 82.55 135.89))
+    (stroke (width 0) (type default))
+  )
+  (wire (pts (xy 87.63 135.89) (xy 87.63 129.54))
+    (stroke (width 0) (type default))
+  )
+  (wire (pts (xy 74.93 101.6) (xy 74.93 95.25))
     (stroke (width 0) (type default))
   )
@@
     (stroke (width 0) (type default))
   )
-  (wire (pts (xy 54.61 110.49) (xy 87.63 101.6))
-    (stroke (width 0) (type default))
-  )
-  (wire (pts (xy 255.27 73.66) (xy 269.24 92.71))
+  (wire (pts (xy 54.61 110.49) (xy 95.25 101.6))
+    (stroke (width 0) (type default))
+  )
+  (wire (pts (xy 255.27 73.66) (xy 276.86 92.71))
     (stroke (width 0) (type default))
   )
@@
     (stroke (width 0) (type default))
   )
-  (wire (pts (xy 54.61 60.96) (xy 74.93 67.31))
+  (wire (pts (xy 54.61 60.96) (xy 82.55 67.31))
     (stroke (width 0) (type default))
   )
@@
     (stroke (width 0) (type default))
   )
-  (wire (pts (xy 54.61 95.25) (xy 74.93 101.6))
-    (stroke (width 0) (type default))
-  )
-  (wire (pts (xy 95.25 168.91) (xy 95.25 162.56))
+  (wire (pts (xy 54.61 95.25) (xy 82.55 101.6))
+    (stroke (width 0) (type default))
+  )
+  (wire (pts (xy 87.63 168.91) (xy 87.63 162.56))
     (stroke (width 0) (type default))
   )
@@
     (stroke (width 0) (type default))
   )
-  (wire (pts (xy 289.56 92.71) (xy 289.56 85.09))
+  (wire (pts (xy 281.94 92.71) (xy 281.94 85.09))
     (stroke (width 0) (type default))
   )
@@
     )
   )
-  (global_label "VBIAS" (shape input) (at 82.55 162.56 0)
-    (effects (font (size 1.27 1.27)) (justify left bottom))
-    (property "Intersheetrefs" "${INTERSHEET_REFS}" (at 82.55 162.56 0)
-      (effects (font (size 1.27 1.27)) hide)
-    )
-  )
-  (global_label "VBIAS" (shape input) (at 95.25 95.25 0)
-    (effects (font (size 1.27 1.27)) (justify left bottom))
-    (property "Intersheetrefs" "${INTERSHEET_REFS}" (at 95.25 95.25 0)
-      (effects (font (size 1.27 1.27)) hide)
-    )
-  )
-  (global_label "VBIAS" (shape input) (at 95.25 60.96 0)
-    (effects (font (size 1.27 1.27)) (justify left bottom))
-    (property "Intersheetrefs" "${INTERSHEET_REFS}" (at 95.25 60.96 0)
-      (effects (font (size 1.27 1.27)) hide)
-    )
-  )
-  (global_label "VBIAS" (shape input) (at 82.55 95.25 0)
-    (effects (font (size 1.27 1.27)) (justify left bottom))
-    (property "Intersheetrefs" "${INTERSHEET_REFS}" (at 82.55 95.25 0)
-      (effects (font (size 1.27 1.27)) hide)
-    )
-  )
-  (global_label "VBIAS" (shape input) (at 289.56 85.09 0)
-    (effects (font (size 1.27 1.27)) (justify left bottom))
-    (property "Intersheetrefs" "${INTERSHEET_REFS}" (at 289.56 85.09 0)
+  (global_label "VBIAS" (shape input) (at 74.93 162.56 0)
+    (effects (font (size 1.27 1.27)) (justify left bottom))
+    (property "Intersheetrefs" "${INTERSHEET_REFS}" (at 74.93 162.56 0)
+      (effects (font (size 1.27 1.27)) hide)
+    )
+  )
+  (global_label "VBIAS" (shape input) (at 87.63 95.25 0)
+    (effects (font (size 1.27 1.27)) (justify left bottom))
+    (property "Intersheetrefs" "${INTERSHEET_REFS}" (at 87.63 95.25 0)
+      (effects (font (size 1.27 1.27)) hide)
+    )
+  )
+  (global_label "VBIAS" (shape input) (at 87.63 60.96 0)
+    (effects (font (size 1.27 1.27)) (justify left bottom))
+    (property "Intersheetrefs" "${INTERSHEET_REFS}" (at 87.63 60.96 0)
+      (effects (font (size 1.27 1.27)) hide)
+    )
+  )
+  (global_label "VBIAS" (shape input) (at 74.93 95.25 0)
+    (effects (font (size 1.27 1.27)) (justify left bottom))
+    (property "Intersheetrefs" "${INTERSHEET_REFS}" (at 74.93 95.25 0)
+      (effects (font (size 1.27 1.27)) hide)
+    )
+  )
+  (global_label "VBIAS" (shape input) (at 281.94 85.09 0)
+    (effects (font (size 1.27 1.27)) (justify left bottom))
+    (property "Intersheetrefs" "${INTERSHEET_REFS}" (at 281.94 85.09 0)
       (effects (font (size 1.27 1.27)) hide)
     )
@@
     )
   )
-  (global_label "VBIAS" (shape input) (at 82.55 129.54 0)
-    (effects (font (size 1.27 1.27)) (justify left bottom))
-    (property "Intersheetrefs" "${INTERSHEET_REFS}" (at 82.55 129.54 0)
+  (global_label "VBIAS" (shape input) (at 74.93 129.54 0)
+    (effects (font (size 1.27 1.27)) (justify left bottom))
+    (property "Intersheetrefs" "${INTERSHEET_REFS}" (at 74.93 129.54 0)
       (effects (font (size 1.27 1.27)) hide)
     )
@@
     )
   )
-  (global_label "VBIAS" (shape input) (at 276.86 85.09 0)
-    (effects (font (size 1.27 1.27)) (justify left bottom))
-    (property "Intersheetrefs" "${INTERSHEET_REFS}" (at 276.86 85.09 0)
-      (effects (font (size 1.27 1.27)) hide)
-    )
-  )
-  (global_label "VBIAS" (shape input) (at 82.55 60.96 0)
-    (effects (font (size 1.27 1.27)) (justify left bottom))
-    (property "Intersheetrefs" "${INTERSHEET_REFS}" (at 82.55 60.96 0)
+  (global_label "VBIAS" (shape input) (at 269.24 85.09 0)
+    (effects (font (size 1.27 1.27)) (justify left bottom))
+    (property "Intersheetrefs" "${INTERSHEET_REFS}" (at 269.24 85.09 0)
+      (effects (font (size 1.27 1.27)) hide)
+    )
+  )
+  (global_label "VBIAS" (shape input) (at 74.93 60.96 0)
+    (effects (font (size 1.27 1.27)) (justify left bottom))
+    (property "Intersheetrefs" "${INTERSHEET_REFS}" (at 74.93 60.96 0)
       (effects (font (size 1.27 1.27)) hide)
     )
@@
     )
   )
-  (global_label "VBIAS" (shape input) (at 95.25 162.56 0)
-    (effects (font (size 1.27 1.27)) (justify left bottom))
-    (property "Intersheetrefs" "${INTERSHEET_REFS}" (at 95.25 162.56 0)
+  (global_label "VBIAS" (shape input) (at 87.63 162.56 0)
+    (effects (font (size 1.27 1.27)) (justify left bottom))
+    (property "Intersheetrefs" "${INTERSHEET_REFS}" (at 87.63 162.56 0)
       (effects (font (size 1.27 1.27)) hide)
     )
@@
     )
   )
-  (global_label "VBIAS" (shape input) (at 95.25 129.54 0)
-    (effects (font (size 1.27 1.27)) (justify left bottom))
-    (property "Intersheetrefs" "${INTERSHEET_REFS}" (at 95.25 129.54 0)
-      (effects (font (size 1.27 1.27)) hide)
-    )
+  (global_label "VBIAS" (shape input) (at 87.63 129.54 0)
+    (effects (font (size 1.27 1.27)) (justify left bottom))
+    (property "Intersheetrefs" "${INTERSHEET_REFS}" (at 87.63 129.54 0)
+      (effects (font (size 1.27 1.27)) hide)
+    )
