File: v2/hardware/KiCad/MeetingHub-4-v2/TRRS.kicad_sch (KiCad schematic)
At the start: 4 parts, among them J2 TRRS Notebook 1, J3 TRRS Notebook 2, J4 TRRS Notebook 3, J5 TRRS Notebook 4

Commit message: V2 corrigida, pronta para produção
Parts:
- J2, J3, J4, J5: footprint MeetingHub-4:Jack_3.5mm_PJ320E_Horizontal -> MeetingHub-4:Jack_3.5mm_PJ-3200B-4A_Horizontal
Changed lines of the file:
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@@
       (effects (font (size 1.27 1.27)))
     )
-    (property "Footprint" "MeetingHub-4:Jack_3.5mm_PJ320E_Horizontal" (at 49.53 77.47 0)
+    (property "Footprint" "MeetingHub-4:Jack_3.5mm_PJ-3200B-4A_Horizontal" (at 49.53 77.47 0)
       (effects (font (size 1.27 1.27)) hide)
     )
@@
       (effects (font (size 1.27 1.27)))
     )
-    (property "Footprint" "MeetingHub-4:Jack_3.5mm_PJ320E_Horizontal" (at 49.53 153.67 0)
+    (property "Footprint" "MeetingHub-4:Jack_3.5mm_PJ-3200B-4A_Horizontal" (at 49.53 153.67 0)
       (effects (font (size 1.27 1.27)) hide)
     )
@@
       (effects (font (size 1.27 1.27)))
     )
-    (property "Footprint" "MeetingHub-4:Jack_3.5mm_PJ320E_Horizontal" (at 49.53 39.37 0)
+    (property "Footprint" "MeetingHub-4:Jack_3.5mm_PJ-3200B-4A_Horizontal" (at 49.53 39.37 0)
       (effects (font (size 1.27 1.27)) hide)
     )
@@
       (effects (font (size 1.27 1.27)))
     )
-    (property "Footprint" "MeetingHub-4:Jack_3.5mm_PJ320E_Horizontal" (at 49.53 115.57 0)
+    (property "Footprint" "MeetingHub-4:Jack_3.5mm_PJ-3200B-4A_Horizontal" (at 49.53 115.57 0)
       (effects (font (size 1.27 1.27)) hide)
     )
