File: v2/hardware/KiCad/MeetingHub-4-v2/HPAMP.kicad_sch (KiCad schematic)
At the start: 17 parts, among them J6 Headset (User), U2 NJM4556A

Commit message: V2 corrigida, pronta para produção
Parts:
- J6: footprint MeetingHub-4:Jack_3.5mm_PJ320E_Horizontal -> MeetingHub-4:Jack_3.5mm_PJ-3200B-4A_Horizontal
Changed lines of the file:
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@@
       (effects (font (size 1.27 1.27)))
     )
-    (property "Footprint" "MeetingHub-4:Jack_3.5mm_PJ320E_Horizontal" (at 199.39 59.69 0)
+    (property "Footprint" "MeetingHub-4:Jack_3.5mm_PJ-3200B-4A_Horizontal" (at 199.39 59.69 0)
       (effects (font (size 1.27 1.27)) hide)
     )

Commit message: Ajuste para não vazar audio, gerada v3 só com microfone
Parts:
- R16, R20: value 47 -> 10
Changed lines of the file:
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@@
       (effects (font (size 1.27 1.27)))
     )
-    (property "Value" "47" (at 165.1 86.36 0)
+    (property "Value" "10" (at 165.1 86.36 0)
       (effects (font (size 1.27 1.27)))
     )
@@
       (effects (font (size 1.27 1.27)))
     )
-    (property "Value" "47" (at 165.1 45.72 0)
-      (effects (font (size 1.27 1.27)))
-    )
+    (property "Value" "10" (at 165.1 45.72 0)
+      (effects (font (size 1.27 1.27)))
+    )
