File: v2/hardware/KiCad/MeetingHub-4-v2/MICSW.kicad_sch (KiCad schematic)
At the start: 8 parts, among them K1 Select NB1, K2 Select NB2, K3 Select NB3, K4 Select NB4

Commit message: Ajuste para não vazar audio, gerada v3 só com microfone
Parts:
- added R39, R40, R41, R42: 2k2, Resistor_THT:R_Axial_DIN0207_L6.3mm_D2.5mm_P10.16mm_Horizontal, symbol Device:R
Connections:
- net HEADSET_MIC: now also K1.10, K2.10, K3.10, K4.10; no longer K1.5, K1.6, K2.5, K2.6, K3.5, K3.6, K4.5, K4.6
- net NB1_MIC: now also K1.5, K1.6; no longer K1.10
- net NB2_MIC: now also K2.5, K2.6; no longer K2.10
- net NB3_MIC: now also K3.5, K3.6; no longer K3.10
- net NB4_MIC: now also K4.5, K4.6; no longer K4.10
- net NCHLD1: now reaches K1.1
- net NCHLD1: now also R39.1
- net NCHLD2: now reaches K2.1
- net NCHLD2: now also R40.1
- net NCHLD3: now reaches K3.1
- net NCHLD3: now also R41.1
- net NCHLD4: now reaches K4.1
- net NCHLD4: now also R42.1
- new net GND: R39.2, R40.2, R41.2, R42.2
- no-connect marks 4 -> 0
