File: v2/hardware/KiCad/MeetingHub-4-v2/SELECT_LOGIC.kicad_sch (KiCad schematic)
At the start: 53 parts, among them Q1 2N7000, Q2 2N7000, Q3 2N7000, Q4 2N7000, SW2 Select NB1 (momentary), SW3 Select NB2 (momentary), SW4 Select NB3 (momentary), SW5 Select NB4 (momentary), U3 LM358, U4 CD4043B

Commit message: V2 corrigida, pronta para produção
Parts:
- SW2, SW3, SW4, SW5: footprint Button_Switch_THT:SW_PUSH_6mm -> Button_Switch_THT:SW_Tactile_SPST_Angled_PTS645Vx39-2LFS
Changed lines of the file:
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@@
     (property "Reference" "SW2" (at 30.48 18.48 0) (effects (font (size 1.27 1.27))))
     (property "Value" "Select NB1 (momentary)" (at 30.48 42.480000000000004 0) (effects (font (size 1.27 1.27))))
-    (property "Footprint" "Button_Switch_THT:SW_PUSH_6mm" (at 30.48 30.48 0) (effects (font (size 1.27 1.27)) hide))
+    (property "Footprint" "Button_Switch_THT:SW_Tactile_SPST_Angled_PTS645Vx39-2LFS" (at 30.48 30.48 0) (effects (font (size 1.27 1.27)) hide))
     (property "Datasheet" "" (at 30.48 30.48 0) (effects (font (size 1.27 1.27)) hide))
     (pin "1")
@@
     (property "Reference" "SW3" (at 30.48 40.07 0) (effects (font (size 1.27 1.27))))
     (property "Value" "Select NB2 (momentary)" (at 30.48 64.07 0) (effects (font (size 1.27 1.27))))
-    (property "Footprint" "Button_Switch_THT:SW_PUSH_6mm" (at 30.48 52.07 0) (effects (font (size 1.27 1.27)) hide))
+    (property "Footprint" "Button_Switch_THT:SW_Tactile_SPST_Angled_PTS645Vx39-2LFS" (at 30.48 52.07 0) (effects (font (size 1.27 1.27)) hide))
     (property "Datasheet" "" (at 30.48 52.07 0) (effects (font (size 1.27 1.27)) hide))
     (pin "1")
@@
     (property "Reference" "SW4" (at 30.48 61.66 0) (effects (font (size 1.27 1.27))))
     (property "Value" "Select NB3 (momentary)" (at 30.48 85.66 0) (effects (font (size 1.27 1.27))))
-    (property "Footprint" "Button_Switch_THT:SW_PUSH_6mm" (at 30.48 73.66 0) (effects (font (size 1.27 1.27)) hide))
+    (property "Footprint" "Button_Switch_THT:SW_Tactile_SPST_Angled_PTS645Vx39-2LFS" (at 30.48 73.66 0) (effects (font (size 1.27 1.27)) hide))
     (property "Datasheet" "" (at 30.48 73.66 0) (effects (font (size 1.27 1.27)) hide))
     (pin "1")
@@
     (property "Reference" "SW5" (at 30.48 84.52 0) (effects (font (size 1.27 1.27))))
     (property "Value" "Select NB4 (momentary)" (at 30.48 108.52 0) (effects (font (size 1.27 1.27))))
-    (property "Footprint" "Button_Switch_THT:SW_PUSH_6mm" (at 30.48 96.52 0) (effects (font (size 1.27 1.27)) hide))
+    (property "Footprint" "Button_Switch_THT:SW_Tactile_SPST_Angled_PTS645Vx39-2LFS" (at 30.48 96.52 0) (effects (font (size 1.27 1.27)) hide))
     (property "Datasheet" "" (at 30.48 96.52 0) (effects (font (size 1.27 1.27)) hide))
     (pin "1")
