File: v2/hardware/KiCad/MeetingHub-4-v2/MeetingHub-4-v2.kicad_pcb (KiCad board)
At the start: 2 copper layers, 192 x 156 mm, 125 parts, among them J1 USB_C_Receptacle_GCT_USB4085, J2 Jack_3.5mm_PJ320E_Horizontal, J3 Jack_3.5mm_PJ320E_Horizontal, J4 Jack_3.5mm_PJ320E_Horizontal, J5 Jack_3.5mm_PJ320E_Horizontal, J6 Jack_3.5mm_PJ320E_Horizontal, K1 Relay_SPDT_Omron_G5V-1, K2 Relay_SPDT_Omron_G5V-1, K3 Relay_SPDT_Omron_G5V-1, K4 Relay_SPDT_Omron_G5V-1, Q1 TO-92_Inline, Q2 TO-92_Inline, Q3 TO-92_Inline, Q4 TO-92_Inline, SW2 SW_PUSH_6mm, SW3 SW_PUSH_6mm, SW4 SW_PUSH_6mm, SW5 SW_PUSH_6mm, U1 DIP-8_W7.62mm, U2 DIP-8_W7.62mm, U3 DIP-8_W7.62mm, U4 DIP-16_W7.62mm

Commit message: V2 corrigida, pronta para produção
Parts:
- J2, J3, J4, J5, J6: value Jack_3.5mm_PJ320E_Horizontal -> Jack_3.5mm_PJ-3200B-4A_Horizontal; footprint MeetingHub-4:Jack_3.5mm_PJ320E_Horizontal -> MeetingHub-4:Jack_3.5mm_PJ-3200B-4A_Horizontal
- SW2, SW3, SW4, SW5: value SW_PUSH_6mm -> SW_Tactile_SPST_Angled_PTS645Vx39-2LFS; footprint Button_Switch_THT:SW_PUSH_6mm -> Button_Switch_THT:SW_Tactile_SPST_Angled_PTS645Vx39-2LFS
- moved SW2 5.00 mm to (124.0, 165.0), turned to 180 degrees
- moved SW3 5.00 mm to (138.0, 165.0), turned to 180 degrees
- moved SW4 5.00 mm to (152.0, 165.0), turned to 180 degrees
- moved SW5 5.00 mm to (166.0, 165.0), turned to 180 degrees
- moved RV1 2.50 mm to (30.0, 162.5)
- moved RV2 2.50 mm to (45.0, 162.5)
- moved RV3 2.50 mm to (60.0, 162.5)
- moved RV4 2.50 mm to (75.0, 162.5)
- moved RV5 2.50 mm to (90.0, 162.5)
- moved J2 1.20 mm to (112.0, 22.2)
- moved J3 1.20 mm to (135.0, 22.2)
- moved J4 1.20 mm to (158.0, 22.2)
- moved J5 1.20 mm to (181.0, 22.2)
- moved J6 0.80 mm to (182.0, 157.8)
Routing:
- net /SELECT_LOGIC/GATE1: track 155.4 -> 118.6 mm, vias 2 -> 1
- net NB2_R: track 170.9 -> 137.9 mm, vias 1 -> 0
- net NB1_R: track 170.0 -> 140.6 mm
- net NB4_R: track 246.2 -> 224.7 mm, vias 1 -> 2
- net NB4_L: track 233.8 -> 252.1 mm
- net Net-(R11-Pad1): track 88.0 -> 103.0 mm, vias 1 -> 0
- net NB1_L: track 182.4 -> 168.1 mm, vias 1 -> 2
- net Net-(R9-Pad1): track 88.8 -> 102.7 mm, vias 0 -> 1
- net Net-(R7-Pad1): track 102.5 -> 88.8 mm, vias 0 -> 1
- net Net-(C20-Pad1): track 40.4 -> 52.2 mm
- net Net-(C16-Pad1): track 88.7 -> 77.3 mm, vias 0 -> 1
- net /SELECT_LOGIC/RST4: track 162.3 -> 152.8 mm, vias 2 -> 0
- net NB3_L: track 181.6 -> 172.8 mm
- net /SELECT_LOGIC/BTN1: track 61.9 -> 70.6 mm
- net NB2_MIC: track 35.2 -> 43.9 mm
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
Commit message: Ajuste para não vazar audio, gerada v3 só com microfone
Parts:
- added R39: R_Axial_DIN0207_L6.3mm_D2.5mm_P10.16mm_Horizontal, Resistor_THT:R_Axial_DIN0207_L6.3mm_D2.5mm_P10.16mm_Horizontal, F.Cu at (168.0, 102.0)
- added R40: R_Axial_DIN0207_L6.3mm_D2.5mm_P10.16mm_Horizontal, Resistor_THT:R_Axial_DIN0207_L6.3mm_D2.5mm_P10.16mm_Horizontal, F.Cu at (168.0, 108.0)
- added R41: R_Axial_DIN0207_L6.3mm_D2.5mm_P10.16mm_Horizontal, Resistor_THT:R_Axial_DIN0207_L6.3mm_D2.5mm_P10.16mm_Horizontal, F.Cu at (168.0, 114.0)
- added R42: R_Axial_DIN0207_L6.3mm_D2.5mm_P10.16mm_Horizontal, Resistor_THT:R_Axial_DIN0207_L6.3mm_D2.5mm_P10.16mm_Horizontal, F.Cu at (168.0, 120.0)
Connections:
- K1 pad 1: (no net) -> /MIC_SWITCHING/NCHLD1
- K1 pad 10: NB1_MIC -> HEADSET_MIC
- K1 pad 5: HEADSET_MIC -> NB1_MIC
- K1 pad 6: HEADSET_MIC -> NB1_MIC
- K2 pad 1: (no net) -> /MIC_SWITCHING/NCHLD2
- K2 pad 10: NB2_MIC -> HEADSET_MIC
- K2 pad 5: HEADSET_MIC -> NB2_MIC
- K2 pad 6: HEADSET_MIC -> NB2_MIC
- K3 pad 1: (no net) -> /MIC_SWITCHING/NCHLD3
- K3 pad 10: NB3_MIC -> HEADSET_MIC
- K3 pad 5: HEADSET_MIC -> NB3_MIC
- K3 pad 6: HEADSET_MIC -> NB3_MIC
- K4 pad 1: (no net) -> /MIC_SWITCHING/NCHLD4
- K4 pad 10: NB4_MIC -> HEADSET_MIC
- K4 pad 5: HEADSET_MIC -> NB4_MIC
- K4 pad 6: HEADSET_MIC -> NB4_MIC
Routing:
- net /MIC_SWITCHING/NCHLD1: track 0.00 -> 88.5 mm, vias 0 -> 1
- net /MIC_SWITCHING/NCHLD3: track 0.00 -> 74.6 mm, vias 0 -> 1
- net /MIC_SWITCHING/NCHLD4: track 0.00 -> 74.3 mm
- net /MIC_SWITCHING/NCHLD2: track 0.00 -> 73.7 mm
- net NB4_L: track 252.1 -> 223.3 mm
- net /SELECT_LOGIC/BTN3: track 115.3 -> 96.1 mm, vias 1 -> 0
- net NB2_R: track 137.9 -> 156.3 mm, vias 0 -> 1
- net /SELECT_LOGIC/RST3: track 187.7 -> 170.6 mm, vias 0 -> 2
- net /SELECT_LOGIC/SET3: track 126.8 -> 110.3 mm, vias 0 -> 1
- net /SELECT_LOGIC/PORN: track 115.4 -> 131.2 mm, vias 3 -> 2
- net MIX_L: track 78.2 -> 62.6 mm, vias 1 -> 0
- net Net-(R9-Pad1): track 102.7 -> 87.3 mm, vias 1 -> 0
- net NB3_MIC: track 35.0 -> 50.2 mm
- net NB4_MIC: track 34.4 -> 49.0 mm
- net /SELECT_LOGIC/BTN1: track 70.6 -> 56.4 mm
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
Commit message: Ajustes footprint para caber j2-j6
Parts:
- moved J2 2.20 mm to (112.0, 20.0)
- moved J3 2.20 mm to (135.0, 20.0)
- moved J4 2.20 mm to (158.0, 20.0)
- moved J5 2.20 mm to (181.0, 20.0)
- moved J6 2.20 mm to (182.0, 160.0)
Routing:
- net COIL4: track 50.2 -> 135.1 mm, vias 0 -> 1
- net NB1_R: track 144.3 -> 175.9 mm
- net /MIC_SWITCHING/NCHLD3: track 74.6 -> 100.4 mm
- net NB4_R: track 227.2 -> 248.6 mm
- net NB2_R: track 156.3 -> 177.3 mm
- net Net-(R11-Pad1): track 89.2 -> 109.6 mm
- net NB3_R: track 160.9 -> 178.9 mm
- net /SELECT_LOGIC/GATE1: track 124.3 -> 140.8 mm, vias 1 -> 2
- net /SELECT_LOGIC/PORN: track 131.2 -> 114.7 mm, vias 2 -> 1
- net Net-(R7-Pad1): track 100.3 -> 85.9 mm
- net Net-(R12-Pad1): track 84.6 -> 98.5 mm, vias 1 -> 0
- net Net-(C14-Pad1): track 126.8 -> 113.1 mm, vias 3 -> 1
- net NB1_L: track 155.4 -> 169.1 mm
- net /SELECT_LOGIC/BTN2: track 74.4 -> 61.3 mm
- net Net-(C10-Pad2): track 71.7 -> 58.6 mm
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